File: controller_mega32l/controller_mega32l.sch (KiCad schematic (older format))
At the start: 81 parts, among them IC1 ATMEGA32-A, IC2 MAX481CPA, J1 RJ45, K1 CONN_PWR_OUT, P1 CONN_PWR_IN, P2 CONN_PWM_OUT, P3 CONN_3X2, P4 CONN_JTAG, P5 CONN_ADC, P6 CONN_GPIO, Q1 NPN

Commit message: PCB signal layer
Parts:
- added J_Network: 3xRJ11, symbol CustomLibrary:3xRJ11
- C1, C2, C3, C4, C5, C6, C7, C8: symbol C-RESCUE-controller_mega32l -> controller_mega32l-rescue:C-RESCUE-controller_mega32l
- D1, D16, D17, D19: symbol ZENER-RESCUE-controller_mega32l -> controller_mega32l-rescue:ZENER-RESCUE-controller_mega32l
- D10, D11, D12, D13, D18, D2, D21, D22, D23, D25, D26, D28, D4, D5, D7, D8: symbol DIODE -> controller_mega32l-rescue:DIODE
- D14, D15, D20, D24, D27, D3, D6, D9: symbol D_Schottky_x2_KCom_AAK -> controller_mega32l-rescue:D_Schottky_x2_KCom_AAK
- IC1: symbol ATMEGA32-A -> controller_mega32l-rescue:ATMEGA32-A
- IC2: symbol MAX481CPA -> controller_mega32l-rescue:MAX481CPA
- J1: symbol RJ45 -> controller_mega32l-rescue:RJ45
- K1: symbol CONN_3 -> controller_mega32l-rescue:CONN_3
- P1: symbol CONN_2 -> controller_mega32l-rescue:CONN_2
- P2, P5: symbol CONN_10 -> controller_mega32l-rescue:CONN_10
- P3: symbol CONN_3X2 -> controller_mega32l-rescue:CONN_3X2
- P4: symbol CONN_5X2 -> controller_mega32l-rescue:CONN_5X2
- P6: symbol CONN_8 -> controller_mega32l-rescue:CONN_8
- Q1: symbol NPN -> controller_mega32l-rescue:NPN
- R1, R10, R11, R12, R13, R14, R15, R16, R17, R18, R19, R2, R20, R21, R22, R23, R24, R25, R26, R27, R28, R29, R3, R30, R31, R32, R33, R34, R4, R5, R6, R7, R8, R9: symbol R-RESCUE-controller_mega32l -> controller_mega32l-rescue:R-RESCUE-controller_mega32l
Connections:
- net DGND: now also J_Network.11, J_Network.14, J_Network.21, J_Network.24, J_Network.31, J_Network.34
- net at D15.2 (A), D18.2 (K), J1.4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: now also J_Network.12, J_Network.22, J_Network.32
- net at D13.2 (K), D15.1 (A), J1.5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: now also J_Network.13, J_Network.23, J_Network.33
Other:
- note added: "RS-485 Alternative Interface"

Commit message: PCB changes
Parts:
- C1: footprint SM1210 -> Capacitor_SMD:C_1210_3225Metric
- C2, C3, C4, C5, C6, C7, C8: footprint SM0805 -> Capacitor_SMD:C_0805_2012Metric
- D1: footprint SM1210L -> Diode_SMD:D_1210_3225Metric
- D10, D11, D12, D13, D14, D15, D18, D2, D23, D24, D25, D26, D27, D28, D3, D4, D5, D6, D7, D8, D9: footprint SOT23 -> digikey-footprints:SOT-23-3
- D20: footprint SM1210L -> digikey-footprints:SOT-23-3
- D21, D22: footprint SM1206 -> digikey-footprints:SOT-23-3
- IC1: footprint TQFP44 -> Package_QFP:TQFP-44_10x10mm_P0.8mm
- IC2: footprint DIP-8__300 -> Package_DIP:DIP-8_W7.62mm
- J1: footprint RJ45_8 -> Connector_RJ:RJ45_Plug_Metz_AJP92A8813
- Q1: footprint TO220 -> Package_TO_SOT_THT:TO-126-3_Vertical
- R1, R13, R14, R17, R19, R20, R23, R25, R26, R27, R29, R3, R30, R32, R34, R4: footprint C1 -> Resistor_THT:R_Axial_DIN0411_L9.9mm_D3.6mm_P15.24mm_Horizontal
- R10, R11, R12, R15, R16, R18, R2, R21, R22, R24, R28, R31, R33, R5, R6, R7, R8, R9: footprint SM0603 -> Resistor_SMD:R_0603_1608Metric
- renumbered J_Network to J_Network1

Commit message: New PCB routes, footprints updated, KiCAD up version to 5.1
Parts:
- C1: footprint Capacitor_SMD:C_1210_3225Metric -> Capacitor_SMD:C_1210_3225Metric_Pad1.33x2.70mm_HandSolder
- C2, C3, C4, C5, C6, C7, C8: footprint Capacitor_SMD:C_0805_2012Metric -> Capacitor_SMD:C_0805_2012Metric_Pad1.18x1.45mm_HandSolder
- D10, D11, D12, D13, D18, D2, D21, D22, D23, D25, D26, D28, D4, D5, D7, D8: footprint digikey-footprints:SOT-23-3 -> Diode_SMD:D_0805_2012Metric_Pad1.15x1.40mm_HandSolder
- K1: footprint PIN_ARRAY_3X1 -> Connector_PinHeader_2.54mm:PinHeader_1x03_P2.54mm_Vertical
- P1: footprint PIN_ARRAY_5x2 -> Connector_PinHeader_2.54mm:PinHeader_1x02_P2.54mm_Vertical
- P2: footprint pin_array_3x2 -> Connector_PinHeader_2.54mm:PinHeader_2x05_P2.54mm_Vertical
- P3: footprint PIN_ARRAY_5x2 -> Connector_PinHeader_2.54mm:PinHeader_2x03_P2.54mm_Vertical
- P4: footprint PIN_ARRAY_5x2 -> Connector_PinHeader_2.54mm:PinHeader_2x05_P2.54mm_Vertical
- P5: footprint pin_array_4x2 -> Connector_PinHeader_2.54mm:PinHeader_2x05_P2.54mm_Vertical
- P6: footprint PIN_ARRAY_2X1 -> Connector_PinHeader_2.54mm:PinHeader_2x04_P2.54mm_Vertical
Changed lines of the file:
@@
 EESchema Schematic File Version 4
-LIBS:controller_mega32l-cache
-EELAYER 29 0
+EELAYER 30 0
 EELAYER END
 $Descr A2 23386 16535
@@
 F 0 "P1" V 3750 5150 40  0000 C CNN
 F 1 "CONN_PWR_IN" V 3850 5150 40  0000 C CNN
-F 2 "PIN_ARRAY_5x2" H 3800 5150 60  0001 C CNN
+F 2 "Connector_PinHeader_2.54mm:PinHeader_1x02_P2.54mm_Vertical" H 3800 5150 60  0001 C CNN
 F 3 "" H 3800 5150 60  0001 C CNN
 	1    3800 5150
@@
 F 0 "K1" V 4350 5750 50  0000 C CNN
 F 1 "CONN_PWR_OUT" V 4450 5750 40  0000 C CNN
-F 2 "PIN_ARRAY_3X1" H 4400 5750 60  0001 C CNN
+F 2 "Connector_PinHeader_2.54mm:PinHeader_1x03_P2.54mm_Vertical" H 4400 5750 60  0001 C CNN
 F 3 "" H 4400 5750 60  0001 C CNN
 	1    4400 5750
@@
 F 0 "P2" V 7500 13000 60  0000 C CNN
 F 1 "CONN_PWM_OUT" V 7600 13000 60  0000 C CNN
-F 2 "pin_array_3x2" H 7550 13000 60  0001 C CNN
+F 2 "Connector_PinHeader_2.54mm:PinHeader_2x05_P2.54mm_Vertical" H 7550 13000 60  0001 C CNN
 F 3 "" H 7550 13000 60  0001 C CNN
 	1    7550 13000
@@
 F 0 "P5" V 12000 5050 60  0000 C CNN
 F 1 "CONN_ADC" V 12100 5050 60  0000 C CNN
-F 2 "pin_array_4x2" H 12050 5050 60  0001 C CNN
+F 2 "Connector_PinHeader_2.54mm:PinHeader_2x05_P2.54mm_Vertical" H 12050 5050 60  0001 C CNN
 F 3 "" H 12050 5050 60  0001 C CNN
 	1    12050 5050
@@
 F 0 "P6" V 15200 9050 60  0000 C CNN
 F 1 "CONN_GPIO" V 15300 9050 60  0000 C CNN
-F 2 "PIN_ARRAY_2X1" H 15250 9050 60  0001 C CNN
+F 2 "Connector_PinHeader_2.54mm:PinHeader_2x04_P2.54mm_Vertical" H 15250 9050 60  0001 C CNN
 F 3 "" H 15250 9050 60  0001 C CNN
 	1    15250 9050
@@
 F 0 "D28" H 14700 8500 40  0000 C CNN
 F 1 "DIODE" H 14700 8300 40  0000 C CNN
-F 2 "digikey-footprints:SOT-23-3" H 14700 8400 60  0001 C CNN
+F 2 "Diode_SMD:D_0805_2012Metric_Pad1.15x1.40mm_HandSolder" H 14700 8400 60  0001 C CNN
 F 3 "" H 14700 8400 60  0001 C CNN
 	1    14700 8400
@@
 F 0 "D26" H 14300 8500 40  0000 C CNN
 F 1 "DIODE" H 14300 8300 40  0000 C CNN
-F 2 "digikey-footprints:SOT-23-3" H 14300 8400 60  0001 C CNN
+F 2 "Diode_SMD:D_0805_2012Metric_Pad1.15x1.40mm_HandSolder" H 14300 8400 60  0001 C CNN
 F 3 "" H 14300 8400 60  0001 C CNN
 	1    14300 8400
@@
 F 0 "D25" H 13900 8500 40  0000 C CNN
 F 1 "DIODE" H 13900 8300 40  0000 C CNN
-F 2 "digikey-footprints:SOT-23-3" H 13900 8400 60  0001 C CNN
+F 2 "Diode_SMD:D_0805_2012Metric_Pad1.15x1.40mm_HandSolder" H 13900 8400 60  0001 C CNN
 F 3 "" H 13900 8400 60  0001 C CNN
 	1    13900 8400
@@
 F 0 "D22" H 13100 8500 40  0000 C CNN
 F 1 "DIODE" H 13100 8300 40  0000 C CNN
-F 2 "digikey-footprints:SOT-23-3" H 13100 8400 60  0001 C CNN
+F 2 "Diode_SMD:D_0805_2012Metric_Pad1.15x1.40mm_HandSolder" H 13100 8400 60  0001 C CNN
 F 3 "" H 13100 8400 60  0001 C CNN
 	1    13100 8400
@@
 F 0 "D23" H 13500 8500 40  0000 C CNN
 F 1 "DIODE" H 13500 8300 40  0000 C CNN
-F 2 "digikey-footprints:SOT-23-3" H 13500 8400 60  0001 C CNN
+F 2 "Diode_SMD:D_0805_2012Metric_Pad1.15x1.40mm_HandSolder" H 13500 8400 60  0001 C CNN
 F 3 "" H 13500 8400 60  0001 C CNN
 	1    13500 8400
@@
 F 0 "D21" H 12700 8500 40  0000 C CNN
 F 1 "DIODE" H 12700 8300 40  0000 C CNN
-F 2 "digikey-footprints:SOT-23-3" H 12700 8400 60  0001 C CNN
+F 2 "Diode_SMD:D_0805_2012Metric_Pad1.15x1.40mm_HandSolder" H 12700 8400 60  0001 C CNN
 F 3 "" H 12700 8400 60  0001 C CNN
 	1    12700 8400
@@
 F 0 "P3" H 9300 9450 50  0000 C CNN
 F 1 "CONN_3X2" V 9300 9250 40  0000 C CNN
-F 2 "PIN_ARRAY_5x2" H 9300 9200 60  0001 C CNN
+F 2 "Connector_PinHeader_2.54mm:PinHeader_2x03_P2.54mm_Vertical" H 9300 9200 60  0001 C CNN
 F 3 "" H 9300 9200 60  0001 C CNN
 	1    9300 9200
@@
 F 0 "C2" H 4450 9250 50  0000 L CNN
 F 1 "1nF" H 4450 9050 50  0000 L CNN
-F 2 "Capacitor_SMD:C_0805_2012Metric" H 4400 9150 60  0001 C CNN
+F 2 "Capacitor_SMD:C_0805_2012Metric_Pad1.18x1.45mm_HandSolder" H 4400 9150 60  0001 C CNN
 F 3 "" H 4400 9150 60  0001 C CNN
 	1    4400 9150
@@
 F 0 "P4" H 11100 9850 60  0000 C CNN
 F 1 "CONN_JTAG" V 11100 9550 50  0000 C CNN
-F 2 "PIN_ARRAY_5x2" H 11100 9550 60  0001 C CNN
+F 2 "Connector_PinHeader_2.54mm:PinHeader_2x05_P2.54mm_Vertical" H 11100 9550 60  0001 C CNN
 F 3 "" H 11100 9550 60  0001 C CNN
 	1    11100 9550
@@
 F 0 "D12" H 11050 7800 40  0000 C CNN
 F 1 "DIODE" H 11050 7600 40  0000 C CNN
-F 2 "digikey-footprints:SOT-23-3" H 11050 7700 60  0001 C CNN
+F 2 "Diode_SMD:D_0805_2012Metric_Pad1.15x1.40mm_HandSolder" H 11050 7700 60  0001 C CNN
 F 3 "" H 11050 7700 60  0001 C CNN
 	1    11050 7700
@@
 F 0 "D11" H 10750 7800 40  0000 C CNN
 F 1 "DIODE" H 10750 7600 40  0000 C CNN
-F 2 "digikey-footprints:SOT-23-3" H 10750 7700 60  0001 C CNN
+F 2 "Diode_SMD:D_0805_2012Metric_Pad1.15x1.40mm_HandSolder" H 10750 7700 60  0001 C CNN
 F 3 "" H 10750 7700 60  0001 C CNN
 	1    10750 7700
@@
 F 0 "D10" H 10450 7800 40  0000 C CNN
 F 1 "DIODE" H 10450 7600 40  0000 C CNN
-F 2 "digikey-footprints:SOT-23-3" H 10450 7700 60  0001 C CNN
+F 2 "Diode_SMD:D_0805_2012Metric_Pad1.15x1.40mm_HandSolder" H 10450 7700 60  0001 C CNN
 F 3 "" H 10450 7700 60  0001 C CNN
 	1    10450 7700
@@
 F 0 "D8" H 10150 7800 40  0000 C CNN
 F 1 "DIODE" H 10150 7600 40  0000 C CNN
-F 2 "digikey-footprints:SOT-23-3" H 10150 7700 60  0001 C CNN
+F 2 "Diode_SMD:D_0805_2012Metric_Pad1.15x1.40mm_HandSolder" H 10150 7700 60  0001 C CNN
 F 3 "" H 10150 7700 60  0001 C CNN
 	1    10150 7700
@@
 F 0 "D7" H 9850 7800 40  0000 C CNN
 F 1 "DIODE" H 9850 7600 40  0000 C CNN
-F 2 "digikey-footprints:SOT-23-3" H 9850 7700 60  0001 C CNN
+F 2 "Diode_SMD:D_0805_2012Metric_Pad1.15x1.40mm_HandSolder" H 9850 7700 60  0001 C CNN
 F 3 "" H 9850 7700 60  0001 C CNN
 	1    9850 7700
@@
 F 0 "D4" H 9250 7800 40  0000 C CNN
 F 1 "DIODE" H 9250 7600 40  0000 C CNN
-F 2 "digikey-footprints:SOT-23-3" H 9250 7700 60  0001 C CNN
+F 2 "Diode_SMD:D_0805_2012Metric_Pad1.15x1.40mm_HandSolder" H 9250 7700 60  0001 C CNN
 F 3 "" H 9250 7700 60  0001 C CNN
 	1    9250 7700
@@
 F 0 "D5" H 9550 7800 40  0000 C CNN
 F 1 "DIODE" H 9550 7600 40  0000 C CNN
-F 2 "digikey-footprints:SOT-23-3" H 9550 7700 60  0001 C CNN
+F 2 "Diode_SMD:D_0805_2012Metric_Pad1.15x1.40mm_HandSolder" H 9550 7700 60  0001 C CNN
 F 3 "" H 9550 7700 60  0001 C CNN
 	1    9550 7700
@@
 F 0 "D2" H 8950 7800 40  0000 C CNN
 F 1 "DIODE" H 8950 7600 40  0000 C CNN
-F 2 "digikey-footprints:SOT-23-3" H 8950 7700 60  0001 C CNN
+F 2 "Diode_SMD:D_0805_2012Metric_Pad1.15x1.40mm_HandSolder" H 8950 7700 60  0001 C CNN
 F 3 "" H 8950 7700 60  0001 C CNN
 	1    8950 7700
@@
 F 0 "C3" H 4750 9250 50  0000 L CNN
 F 1 "0.1uF" H 4750 9050 50  0000 L CNN
-F 2 "Capacitor_SMD:C_0805_2012Metric" H 4700 9150 60  0001 C CNN
+F 2 "Capacitor_SMD:C_0805_2012Metric_Pad1.18x1.45mm_HandSolder" H 4700 9150 60  0001 C CNN
 F 3 "" H 4700 9150 60  0001 C CNN
 	1    4700 9150
@@
 F 0 "D18" H 12050 12050 40  0000 C CNN
 F 1 "DIODE" H 12050 11850 40  0000 C CNN
-F 2 "digikey-footprints:SOT-23-3" H 12050 11950 60  0001 C CNN
+F 2 "Diode_SMD:D_0805_2012Metric_Pad1.15x1.40mm_HandSolder" H 12050 11950 60  0001 C CNN
 F 3 "" H 12050 11950 60  0001 C CNN
 	1    12050 11950
@@
 F 0 "D13" H 11150 12050 40  0000 C CNN
 F 1 "DIODE" H 11150 11850 40  0000 C CNN
-F 2 "digikey-footprints:SOT-23-3" H 11150 11950 60  0001 C CNN
+F 2 "Diode_SMD:D_0805_2012Metric_Pad1.15x1.40mm_HandSolder" H 11150 11950 60  0001 C CNN
 F 3 "" H 11150 11950 60  0001 C CNN
 	1    11150 11950
@@
 F 0 "C5" H 5300 5650 50  0000 L CNN
 F 1 "0.1uF" H 5300 5450 50  0000 L CNN
-F 2 "Capacitor_SMD:C_0805_2012Metric" H 5250 5550 60  0001 C CNN
+F 2 "Capacitor_SMD:C_0805_2012Metric_Pad1.18x1.45mm_HandSolder" H 5250 5550 60  0001 C CNN
 F 3 "" H 5250 5550 60  0001 C CNN
 	1    5250 5550
@@
 F 0 "C8" H 5300 6550 50  0000 L CNN
 F 1 "0.1uF" H 5300 6350 50  0000 L CNN
-F 2 "Capacitor_SMD:C_0805_2012Metric" H 5250 6450 60  0001 C CNN
+F 2 "Capacitor_SMD:C_0805_2012Metric_Pad1.18x1.45mm_HandSolder" H 5250 6450 60  0001 C CNN
 F 3 "" H 5250 6450 60  0001 C CNN
 	1    5250 6450
@@
 F 0 "C7" H 5300 6250 50  0000 L CNN
 F 1 "0.1uF" H 5300 6050 50  0000 L CNN
-F 2 "Capacitor_SMD:C_0805_2012Metric" H 5250 6150 60  0001 C CNN
+F 2 "Capacitor_SMD:C_0805_2012Metric_Pad1.18x1.45mm_HandSolder" H 5250 6150 60  0001 C CNN
 F 3 "" H 5250 6150 60  0001 C CNN
 	1    5250 6150
@@
 F 0 "C6" H 5300 5950 50  0000 L CNN
 F 1 "0.1uF" H 5300 5750 50  0000 L CNN
-F 2 "Capacitor_SMD:C_0805_2012Metric" H 5250 5850 60  0001 C CNN
+F 2 "Capacitor_SMD:C_0805_2012Metric_Pad1.18x1.45mm_HandSolder" H 5250 5850 60  0001 C CNN
 F 3 "" H 5250 5850 60  0001 C CNN
 	1    5250 5850
@@
 F 0 "C4" H 4800 7800 50  0000 L CNN
 F 1 "1nF" H 4800 7600 50  0000 L CNN
-F 2 "Capacitor_SMD:C_0805_2012Metric" H 4750 7700 60  0001 C CNN
+F 2 "Capacitor_SMD:C_0805_2012Metric_Pad1.18x1.45mm_HandSolder" H 4750 7700 60  0001 C CNN
 F 3 "" H 4750 7700 60  0001 C CNN
 	1    4750 7700
@@
 F 0 "C1" H 3950 7100 50  0000 L CNN
 F 1 "10uF" H 3950 6900 50  0000 L CNN
-F 2 "Capacitor_SMD:C_1210_3225Metric" H 3900 7000 60  0001 C CNN
+F 2 "Capacitor_SMD:C_1210_3225Metric_Pad1.33x2.70mm_HandSolder" H 3900 7000 60  0001 C CNN
 F 3 "" H 3900 7000 60  0001 C CNN
 	1    3900 7000

Commit message: RJ-45 footprint updated, PCB screenshot added to docs
Parts:
- J1: footprint Connector_RJ:RJ45_Plug_Metz_AJP92A8813 -> Connector_RJ:RJ45_Amphenol_54602-x08_Horizontal
Changed lines of the file:
@@
 F 0 "J1" H 13050 11250 60  0000 C CNN
 F 1 "RJ45" H 12700 11250 60  0000 C CNN
-F 2 "Connector_RJ:RJ45_Plug_Metz_AJP92A8813" H 12850 10750 60  0001 C CNN
+F 2 "Connector_RJ:RJ45_Amphenol_54602-x08_Horizontal" H 12850 10750 60  0001 C CNN
 F 3 "" H 12850 10750 60  0001 C CNN
 	1    12850 10750

Commit message: RJ-45 ground connections fixed, PCB texts placed right
Parts:
- C1: footprint Capacitor_SMD:C_1210_3225Metric_Pad1.33x2.70mm_HandSolder -> SM1210
- C2, C3, C4, C5, C6, C7, C8: footprint Capacitor_SMD:C_0805_2012Metric_Pad1.18x1.45mm_HandSolder -> SM0805
- D1: footprint Diode_SMD:D_1210_3225Metric -> SM1210L
- D10, D11, D12, D13, D18, D2, D23, D25, D26, D28, D4, D5, D7, D8: footprint Diode_SMD:D_0805_2012Metric_Pad1.15x1.40mm_HandSolder -> SOT23
- D14, D15, D24, D27, D3, D6, D9: footprint digikey-footprints:SOT-23-3 -> SOT23
- D20: footprint digikey-footprints:SOT-23-3 -> SM1210L
- D21, D22: footprint Diode_SMD:D_0805_2012Metric_Pad1.15x1.40mm_HandSolder -> SM1206
- IC1: footprint Package_QFP:TQFP-44_10x10mm_P0.8mm -> TQFP44
- IC2: footprint Package_DIP:DIP-8_W7.62mm -> DIP-8__300
- J1: footprint Connector_RJ:RJ45_Amphenol_54602-x08_Horizontal -> RJ45_8
- K1: footprint Connector_PinHeader_2.54mm:PinHeader_1x03_P2.54mm_Vertical -> PIN_ARRAY_3X1
- P1: footprint Connector_PinHeader_2.54mm:PinHeader_1x02_P2.54mm_Vertical -> PIN_ARRAY_5x2
- P2: footprint Connector_PinHeader_2.54mm:PinHeader_2x05_P2.54mm_Vertical -> pin_array_3x2
- P3: footprint Connector_PinHeader_2.54mm:PinHeader_2x03_P2.54mm_Vertical -> PIN_ARRAY_5x2
- P4: footprint Connector_PinHeader_2.54mm:PinHeader_2x05_P2.54mm_Vertical -> PIN_ARRAY_5x2
- P5: footprint Connector_PinHeader_2.54mm:PinHeader_2x05_P2.54mm_Vertical -> pin_array_4x2
- P6: footprint Connector_PinHeader_2.54mm:PinHeader_2x04_P2.54mm_Vertical -> PIN_ARRAY_2X1
- Q1: footprint Package_TO_SOT_THT:TO-126-3_Vertical -> TO220
- R1, R13, R14, R17, R19, R20, R23, R25, R26, R27, R29, R3, R30, R32, R34, R4: footprint Resistor_THT:R_Axial_DIN0411_L9.9mm_D3.6mm_P15.24mm_Horizontal -> C1
- R10, R11, R12, R15, R16, R18, R2, R21, R22, R24, R28, R31, R33, R5, R6, R7, R8, R9: footprint Resistor_SMD:R_0603_1608Metric -> SM0603
Connections:
- net DGND: no longer J1.9 (SHIELD), J_Network1.11, J_Network1.14, J_Network1.21, J_Network1.24, J_Network1.31, J_Network1.34
- net at J1.1: now also J1.8, J1.9 (SHIELD), J_Network1.11, J_Network1.14, J_Network1.21, J_Network1.24, J_Network1.31, J_Network1.34, R34.1
